File: hardware/GameOfShrooms2023/GameOfShrooms2023.kicad_pcb (KiCad board)
At the start: 2 copper layers, 62.2 x 86 mm, 27 parts, among them U1 74AHC1G125

Commit message: Exported Gerbers
Routing:
- net GND: track 390.6 -> 379.3 mm
- net +5V: track 184.3 -> 191.4 mm
- net Net-(LED1-DOU): track 16.5 -> 15.4 mm
- net Net-(LED1-DIN): track 9.77 -> 10.3 mm
Other:
- board text added: "@Funvill 2023"
- board text added: "GameOfShrooms"
